File: hardware/atmega328pb_V2_breakout/atmega328pb_v2_breakout/atmega328pb_v2_breakout.kicad_sch (KiCad schematic)
At the start: 23 parts, among them J1 AVR-ISP-6, J2 Conn_01x15_Male, J3 Conn_01x15_Male, J4 Conn_01x06_Male, SW1 SW_Push, U1 ATmega328PB-A, U2 LP2985-5.0, Y1 16MHz

Commit message: Added slimmer version of breakout
Parts:
- removed C2, C3: 22pF, Capacitor_SMD:C_0603_1608Metric_Pad1.08x0.95mm_HandSolder, symbol Device:C_Small
- removed Y1: 16MHz, Crystal:Crystal_SMD_TXC_7A-2Pin_5x3.2mm, symbol Device:Crystal_Small
- added Y1: 16MHz, Crystal:Resonator_SMD_Murata_CSTxExxV-3Pin_3.0x1.1mm, symbol Device:Resonator_Small
- D1: value LED -> PWR; footprint LED_SMD:LED_1206_3216Metric_Pad1.42x1.75mm_HandSolder -> LED_SMD:LED_0805_2012Metric
- D2: value LED -> D13; footprint LED_SMD:LED_1206_3216Metric_Pad1.42x1.75mm_HandSolder -> LED_SMD:LED_0805_2012Metric
- SW1: footprint Button_Switch_THT:SW_PUSH_6mm -> Button_Switch_SMD:SW_SPST_B3U-1000P
Connections:
- net GND: now also Y1.2
- net at U1.7 (XTAL1/PB6): now also Y1.3
- net at U1.8 (XTAL2/PB7): now also Y1.1
