File: hardware/atmega328pb_breakout/atmega328pb_breakout.kicad_pcb (KiCad board)
At the start: 2 copper layers, 21.8 x 42.2 mm, 23 parts, among them J2 Conn_01x15_Male, J3 Conn_01x15_Male, J4 Conn_01x06_Male, SW1 SW_Push, U1 ATmega328P, U2 LP2985, Y1 16MHz

Commit message: Added slimmer version of breakout
Parts:
- U1: value ATmega328P -> ATmega328PB-A
- U2: value LP2985 -> LP2985-5.0
- renumbered POWER to D1, D13 to D2, ISP to J1
Changed lines of the file:
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@@
       (outputformat 1)
       (mirror false)
-      (drillshape 1)
+      (drillshape 0)
       (scaleselection 1)
-      (outputdirectory "")
+      (outputdirectory "../../production/gerbers/")
     )
   )
@@
       (effects (font (size 1 1) (thickness 0.15)))
     )
-    (fp_text value "Conn_01x15_Male" (at 0 37.89) (layer "F.Fab")
+    (fp_text value "Conn_01x15_Male" (at 3.302 30.48 90) (layer "F.Fab")
       (effects (font (size 1 1) (thickness 0.15)))
     )
@@
       (effects (font (size 1 1) (thickness 0.15)))
     )
-    (fp_text value "ATmega328P" (at -0.179605 0.179605 180) (layer "F.SilkS")
+    (fp_text value "ATmega328PB-A" (at -0.179605 0.179605 180) (layer "F.SilkS")
       (effects (font (size 0.5 0.5) (thickness 0.075)))
     )
@@
     (property "Sheetname" "")
     (attr smd)
-    (fp_text reference "D13" (at -0.2175 1.778 -90) (layer "F.SilkS")
+    (fp_text reference "D2" (at -0.2175 1.778 -90) (layer "F.SilkS")
       (effects (font (size 0.75 0.75) (thickness 0.1)))
     )
@@
     (fp_line (start 1.6 0.8) (end 1.6 -0.8) (layer "F.Fab") (width 0.1))
     (fp_line (start -1.2 -0.8) (end -1.6 -0.4) (layer "F.Fab") (width 0.1))
-    (pad "1" smd roundrect (at -1.4875 0 270) (size 1.425 1.75) (layers "F.Cu" "F.Paste" "F.Mask") (roundrect_rratio 0.175439)
+    (pad "1" smd roundrect (at -1.4875 0 270) (size 1.425 1.75) (layers "F.Cu" "F.Paste" "F.Mask") (roundrect_rratio 0.1754392982)
       (net 36 "Net-(D2-Pad1)") (pinfunction "K") (pintype "passive"))
-    (pad "2" smd roundrect (at 1.4875 0 270) (size 1.425 1.75) (layers "F.Cu" "F.Paste" "F.Mask") (roundrect_rratio 0.175439)
+    (pad "2" smd roundrect (at 1.4875 0 270) (size 1.425 1.75) (layers "F.Cu" "F.Paste" "F.Mask") (roundrect_rratio 0.1754392982)
       (net 10 "D13") (pinfunction "A") (pintype "passive"))
     (model "${KICAD6_3DMODEL_DIR}/LED_SMD.3dshapes/LED_1206_3216Metric.wrl"
@@
       (effects (font (size 1 1) (thickness 0.15)))
     )
-    (fp_text value "Conn_01x15_Male" (at 0 38.608) (layer "F.Fab")
+    (fp_text value "Conn_01x15_Male" (at -3.302 30.48 90) (layer "F.Fab")
       (effects (font (size 1 1) (thickness 0.15)))
     )
@@
     (fp_line (start 1 0.45) (end -1 0.45) (layer "F.Fab") (width 0.1))
     (fp_line (start -1 0.45) (end -1 -0.45) (layer "F.Fab") (width 0.1))
-    (pad "1" smd roundrect (at -1.15 0 270) (size 1.05 1.2) (layers "F.Cu" "F.Paste" "F.Mask") (roundrect_rratio 0.238095)
+    (pad "1" smd roundrect (at -1.15 0 270) (size 1.05 1.2) (layers "F.Cu" "F.Paste" "F.Mask") (roundrect_rratio 0.2380952381)
       (net 5 "VDD") (pintype "passive"))
-    (pad "2" smd roundrect (at 1.15 0 270) (size 1.05 1.2) (layers "F.Cu" "F.Paste" "F.Mask") (roundrect_rratio 0.238095)
+    (pad "2" smd roundrect (at 1.15 0 270) (size 1.05 1.2) (layers "F.Cu" "F.Paste" "F.Mask") (roundrect_rratio 0.2380952381)
       (net 2 "VDDA") (pintype "passive"))
     (model "${KICAD6_3DMODEL_DIR}/Inductor_SMD.3dshapes/L_0805_2012Metric.wrl"
@@
       (effects (font (size 0.5 0.5) (thickness 0.075)))
     )
-    (fp_text value "LP2985" (at 0 0.066 90) (layer "F.SilkS")
+    (fp_text value "LP2985-5.0" (at 0 0.066 90) (layer "F.SilkS")
       (effects (font (size 0.5 0.5) (thickness 0.075)))
     )
@@
     (property "Sheetname" "")
     (attr through_hole)
-    (fp_text reference "ISP" (at 0 -2.032) (layer "F.SilkS")
-      (effects (font (size 1 1) (thickness 0.15)))
-    )
-    (fp_text value "AVR-ISP-6" (at 1.27 7.41) (layer "F.Fab")
+    (fp_text reference "J1" (at 0 -2.032) (layer "F.SilkS")
+      (effects (font (size 1 1) (thickness 0.15)))
+    )
+    (fp_text value "AVR-ISP-6" (at 1.016 7.874) (layer "F.Fab")
       (effects (font (size 1 1) (thickness 0.15)))
     )
@@
     (property "Sheetname" "")
     (attr smd)
-    (fp_text reference "POWER" (at 0 1.778 90) (layer "F.SilkS")
+    (fp_text reference "D1" (at 0 1.778 90) (layer "F.SilkS")
       (effects (font (size 0.75 0.75) (thickness 0.1)))
     )
@@
     (fp_line (start -1.6 0.8) (end 1.6 0.8) (layer "F.Fab") (width 0.1))
     (fp_line (start 1.6 -0.8) (end -1.2 -0.8) (layer "F.Fab") (width 0.1))
-    (pad "1" smd roundrect (at -1.4875 0 270) (size 1.425 1.75) (layers "F.Cu" "F.Paste" "F.Mask") (roundrect_rratio 0.175439)
+    (pad "1" smd roundrect (at -1.4875 0 270) (size 1.425 1.75) (layers "F.Cu" "F.Paste" "F.Mask") (roundrect_rratio 0.1754392982)
       (net 35 "Net-(D1-Pad1)") (pinfunction "K") (pintype "passive"))
-    (pad "2" smd roundrect (at 1.4875 0 270) (size 1.425 1.75) (layers "F.Cu" "F.Paste" "F.Mask") (roundrect_rratio 0.175439)
+    (pad "2" smd roundrect (at 1.4875 0 270) (size 1.425 1.75) (layers "F.Cu" "F.Paste" "F.Mask") (roundrect_rratio 0.1754392982)
       (net 5 "VDD") (pinfunction "A") (pintype "passive"))
     (model "${KICAD6_3DMODEL_DIR}/LED_SMD.3dshapes/LED_1206_3216Metric.wrl"
